Commit message: feat(kinematics): OBB box proxy + stack neck-segment URDF origins
- proxies.py: box primitives now map to an oriented bounding Box (OBB)
  faithfully enclosing flat slabs, replacing the over-enclosing capsule/
  sphere box rule that swelled the torso into a fat cylinder
- collision.py: add sphere_box/capsule_box/box_box (SAT) distance fns +
  Box world-placement and pair dispatch
- maximus.urdf: give lower_neck_joint (z=0.046) and pitch_neck_joint
  (z=0.014) their true vertical offsets so neck cylinders stack instead
  of piling up coincident at z=0.275
- design.md: document the OBB proxy + box distance functions
- test_proxies.py: box->Box assertions; Box branches in enclosure/monotonic
  property tests

File: src/config/maximus.urdf (robot description, URDF)
Before this commit: robot maximus, 10 links, 9 joints
Joints:
- joint lower_neck_joint: origin xyz=0 0 0 rpy=0 0 0 -> xyz=0 0 0.046 rpy=0 0 0
- joint pitch_neck_joint: origin xyz=0 0 0 rpy=0 0 0 -> xyz=0 0 0.014 rpy=0 0 0

Commit message: fix(kinematics): correct arm geometry from measurements + arm self-exempt group
Measured the physical arm and reconciled the URDF, which was substantially off:
- Upper arm 0.19->0.25 m and elbow_yaw_joint origin 0->0.25 (the forearm was
  collapsed onto the shoulder because the elbow joint never advanced along the
  upper arm -- same class of bug as the neck coincidence).
- Forearm 0.17->0.18 m; hand modeled with a ~50deg curl (rpy pitch 0.873) so
  the proxy reaches where the real curled hand reaches (~8 cm closer).
- Shoulder-tilt joint moved out to x=0.1975 (6.5 cm gap from the torso edge;
  it was mounted flush, giving the arm no torso clearance).
- Elbow-tilt scale refit to the right-angle landmark (servo 145 = 90deg bend):
  sign=1 offset=5 scale=0.6429 (was 0.5294, under-bending the forearm).
- Add an arm-segment self-exempt group (upper_arm/elbow/lower_arm) so the
  near-collinear upper-arm vs forearm no longer reads as a false collision when
  the elbow is straight; they still collide normally vs torso/head/neck.
- Update test collision fixtures to a genuine collision (elbow fully flexed
  folds the hand onto the shoulder) instead of the old collinear false positive.

Common poses (rest, arm out, arm up, elbow flexed in open space) classify
SAFE; fully-flexed elbow at the side correctly flags hand<->shoulder.

File: src/config/maximus.urdf (robot description, URDF)
Before this commit: robot maximus, 10 links, 9 joints
Links:
- link lower_arm_link: geometry visual cylinder length=0.18 radius=0.015
- link upper_arm_link: geometry visual cylinder length=0.25 radius=0.015
Joints:
- joint elbow_pitch_joint: origin xyz=0 0 0.285 rpy=0 0 0 -> xyz=0 0 0 rpy=0 0 0
- joint elbow_yaw_joint: origin xyz=0 0 0 rpy=0 0 0 -> xyz=0 0 0.25 rpy=0 0 0
- joint shoulder_yaw_joint: origin xyz=0.1325 0 0.250 rpy=0 0 0 -> xyz=0.1975 0 0.250 rpy=0 0 0
- joint wrist_joint: origin xyz=0 0 0.17 rpy=0 0 0 -> xyz=0 0 0.18 rpy=0 0 0

Commit message: fix(kinematics): model head as an oriented box instead of a sphere
Measured head is oval, not spherical: x=0.08 (front-back depth), y=0.18
(ear-to-ear), z=0.105 (height), centered at world z=0.48. A sphere (r=0.105)
over-reported the shallow front-back axis by ~2x; the box matches the real
head far better. head_link origin is at z=0.505, so the box visual sits 0.025
below it. make_proxy already turns boxes into oriented-box proxies.

File: src/config/maximus.urdf (robot description, URDF)
Before this commit: robot maximus, 10 links, 9 joints
Links:
- link head_link: geometry visual box size=0.08 0.18 0.105
